Commit message: Update crawling-panther.urdf

File: crawling-panther.urdf (robot description, URDF)
Before this commit: robot robot, 11 links, 10 joints
Links:
- link base_link: mass 0.06 -> 0.075; geometry collision box size=0.116 0.1262 0.01; visual box size=0.116 0.1262 0.01
- link extra_box: geometry collision box size=0.065 0.035 0.01; visual box size=0.065 0.035 0.01
- link hip1: geometry collision box size=0.02 0.049 0.03; visual box size=0.02 0.049 0.03
- link hip2: geometry collision box size=0.02 0.049 0.03; visual box size=0.02 0.049 0.03
- link hip3: geometry collision box size=0.02 0.049 0.03; visual box size=0.02 0.049 0.03
- link hip4: geometry collision box size=0.02 0.049 0.03; visual box size=0.02 0.049 0.03
- link leg1: geometry collision box size=0.0205 0.01 0.01; collision box size=0.0479 0.019 0.0095
- link leg2: geometry collision box size=0.0205 0.01 0.01; collision box size=0.0479 0.019 0.0095
- link leg3: geometry collision box size=0.0205 0.01 0.01; collision box size=0.0479 0.019 0.0095
- link leg4: geometry collision box size=0.0205 0.01 0.01; collision box size=0.0479 0.019 0.0095
Joints:
- joint base_joint: origin xyz=0 0 0.5 rpy=0 0 0 -> xyz=0 0 0.05 rpy=0 0 0
- joint base_link_to_extra_box: origin xyz=-0.285 0 0.1 rpy=0 0 1.570796 -> xyz=-0.0285 0 0.01 rpy=0 0 1.570796
- joint base_link_to_hip1: limit lower=-1 upper=1 effort=1000.0 velocity=0.5 -> lower=-1 upper=1 effort=10.0 velocity=5.0; origin xyz=0.365 -0.515 0.1 rpy=0 0 0 -> xyz=0.0365 -0.0515 0.01 rpy=0 0 0
- joint base_link_to_hip2: limit lower=-1 upper=1 effort=1000.0 velocity=0.5 -> lower=-1 upper=1 effort=10.0 velocity=5.0; origin xyz=-0.365 -0.515 0.1 rpy=0 0 0 -> xyz=-0.0365 -0.0515 0.01 rpy=0 0 0
- joint base_link_to_hip3: limit lower=-1 upper=1 effort=1000.0 velocity=0.5 -> lower=-1 upper=1 effort=10.0 velocity=5.0; origin xyz=0.365 0.515 0.1 rpy=0 0 0 -> xyz=0.0365 0.0515 0.01 rpy=0 0 0
- joint base_link_to_hip4: limit lower=-1 upper=1 effort=1000.0 velocity=0.5 -> lower=-1 upper=1 effort=10.0 velocity=5.0; origin xyz=-0.365 0.515 0.1 rpy=0 0 0 -> xyz=-0.0365 0.0515 0.01 rpy=0 0 0
- joint base_link_to_leg1: limit lower=-1 upper=1 effort=1000.0 velocity=0.5 -> lower=-1 upper=1 effort=10.0 velocity=5.0; origin xyz=0.1 -0.405 -0.1 rpy=0 1.5707963267948966 0 -> xyz=0.01 -0.0405 -0.01 rpy=0 1.5707963 0
- joint base_link_to_leg2: limit lower=-1 upper=1 effort=1000.0 velocity=0.5 -> lower=-1 upper=1 effort=10.0 velocity=5.0; origin xyz=-0.1 -0.41 -0.1 rpy=0 1.5707963267948966 0 -> xyz=-0.01 -0.041 -0.01 rpy=0 1.5707963 0
- joint base_link_to_leg3: limit lower=-1 upper=1 effort=1000.0 velocity=0.5 -> lower=-1 upper=1 effort=10.0 velocity=5.0; origin xyz=0.1 0.41 -0.1 rpy=0 1.5707963267948966 0 -> xyz=0.01 0.041 -0.01 rpy=0 1.5707963 0
- joint base_link_to_leg4: limit lower=-1 upper=1 effort=1000.0 velocity=0.5 -> lower=-1 upper=1 effort=10.0 velocity=5.0; origin xyz=-0.1 0.41 -0.1 rpy=0 1.5707963267948966 0 -> xyz=-0.01 0.041 -0.01 rpy=0 1.5707963 0
